File: imu.kicad_sch (KiCad schematic)
At the start: 4 parts, among them IC1 ICM-42688-P

Commit message: Dodano brakujące footprinty do układu wejściowego i poprawiono SPI - zamieniono SCK <-> MISO (na poprawne)
Connections:
- net MISO_imu: now also IC1.1 (AP_SDO_/_AP_AD0); no longer IC1.13 (AP_SCL_/_AP_SCLK)
- net SCK_imu: now also IC1.13 (AP_SCL_/_AP_SCLK); no longer IC1.1 (AP_SDO_/_AP_AD0)
Changed lines of the file:
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@@
+	(wire
+		(pts
+			(xy 90.17 97.79) (xy 109.22 97.79)
+		)
+		(stroke
+			(width 0)
+			(type default)
+		)
+	)
 	(wire
 		(pts
@@
 	(wire
 		(pts
+			(xy 142.24 50.8) (xy 142.24 54.61)
+		)
+		(stroke
+			(width 0)
+			(type default)
+		)
+	)
+	(wire
+		(pts
 			(xy 87.63 100.33) (xy 87.63 102.87)
 		)
@@
 	(wire
 		(pts
-			(xy 142.24 50.8) (xy 142.24 54.61)
-		)
-		(stroke
-			(width 0)
-			(type default)
-		)
-	)
-	(wire
-		(pts
 			(xy 129.54 132.08) (xy 129.54 133.35)
 		)
@@
 		(pts
 			(xy 193.04 113.03) (xy 193.04 114.3)
-		)
-		(stroke
-			(width 0)
-			(type default)
-		)
-	)
-	(wire
-		(pts
-			(xy 90.17 97.79) (xy 109.22 97.79)
 		)
 		(stroke
@@
 	(text "PRZED USTALENIEM POZYCJI NA PCB\nZAPOZNAĆ SIĘ Z DOKUMENTACJĄ UKŁADU!!!"
 		(exclude_from_sim no)
-		(at 205.232 36.83 0)
+		(at 238.506 21.59 0)
 		(effects
 			(font
@@
 	(hierarchical_label "MISO_imu"
 		(shape output)
-		(at 142.24 50.8 90)
-		(fields_autoplaced yes)
-		(effects
-			(font
-				(size 1.27 1.27)
-			)
-			(justify left)
+		(at 90.17 97.79 180)
+		(fields_autoplaced yes)
+		(effects
+			(font
+				(size 1.27 1.27)
+			)
+			(justify right)
 		)
 	)
 	(hierarchical_label "SCK_imu"
 		(shape input)
-		(at 90.17 97.79 180)
-		(fields_autoplaced yes)
-		(effects
-			(font
-				(size 1.27 1.27)
-			)
-			(justify right)
-		)
-	)
+		(at 142.24 50.8 90)
+		(fields_autoplaced yes)
+		(effects
+			(font
+				(size 1.27 1.27)
+			)
+			(justify left)
+		)
+	)

Commit message: dodano komentarze do projektu
Parts:
- added R17: 10k, Resistor_SMD:R_0603_1608Metric, symbol Device:R
Connections:
- net 3,3V_stm32: now also R17.2
- net CS_imu: now also R17.1
Other:
- note added: "SPRAWDZIĆ CZY JEST OK (rezystor) I CZY MUSI BYC NA MISO (napewno nie ale z jakiegos powodu tak jest teraz fizycznie)"
Changed lines of the file:
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@@
+	)
+	(junction
+		(at 144.78 49.53)
+		(diameter 0)
+		(color 0 0 0 0)
 	)
 	(junction
@@
 	(wire
 		(pts
-			(xy 144.78 50.8) (xy 144.78 54.61)
+			(xy 144.78 45.72) (xy 144.78 49.53)
 		)
 		(stroke
@@
 	(wire
 		(pts
+			(xy 109.22 102.87) (xy 87.63 102.87)
+		)
+		(stroke
+			(width 0)
+			(type default)
+		)
+	)
+	(wire
+		(pts
+			(xy 175.26 100.33) (xy 204.47 100.33)
+		)
+		(stroke
+			(width 0)
+			(type default)
+		)
+	)
+	(wire
+		(pts
+			(xy 144.78 123.19) (xy 144.78 124.46)
+		)
+		(stroke
+			(width 0)
+			(type default)
+		)
+	)
+	(wire
+		(pts
+			(xy 144.78 124.46) (xy 142.24 124.46)
+		)
+		(stroke
+			(width 0)
+			(type default)
+		)
+	)
+	(wire
+		(pts
+			(xy 144.78 49.53) (xy 147.32 49.53)
+		)
+		(stroke
+			(width 0)
+			(type default)
+		)
+	)
+	(wire
+		(pts
+			(xy 144.78 49.53) (xy 144.78 54.61)
+		)
+		(stroke
+			(width 0)
+			(type default)
+		)
+	)
+	(wire
+		(pts
+			(xy 204.47 97.79) (xy 175.26 97.79)
+		)
+		(stroke
+			(width 0)
+			(type default)
+		)
+	)
+	(wire
+		(pts
+			(xy 175.26 105.41) (xy 177.8 105.41)
+		)
+		(stroke
+			(width 0)
+			(type default)
+		)
+	)
+	(wire
+		(pts
+			(xy 129.54 124.46) (xy 125.73 124.46)
+		)
+		(stroke
+			(width 0)
+			(type default)
+		)
+	)
+	(wire
+		(pts
+			(xy 204.47 100.33) (xy 204.47 101.6)
+		)
+		(stroke
+			(width 0)
+			(type default)
+		)
+	)
+	(wire
+		(pts
+			(xy 142.24 45.72) (xy 142.24 54.61)
+		)
+		(stroke
+			(width 0)
+			(type default)
+		)
+	)
+	(wire
+		(pts
+			(xy 87.63 100.33) (xy 87.63 102.87)
+		)
+		(stroke
+			(width 0)
+			(type default)
+		)
+	)
+	(wire
+		(pts
+			(xy 177.8 105.41) (xy 193.04 105.41)
+		)
+		(stroke
+			(width 0)
+			(type default)
+		)
+	)
+	(wire
+		(pts
+			(xy 129.54 132.08) (xy 129.54 133.35)
+		)
+		(stroke
+			(width 0)
+			(type default)
+		)
+	)
+	(wire
+		(pts
+			(xy 33.02 30.48) (xy 45.72 30.48)
+		)
+		(stroke
+			(width 0)
+			(type default)
+		)
+	)
+	(wire
+		(pts
 			(xy 90.17 97.79) (xy 109.22 97.79)
 		)
@@
 	(wire
 		(pts
-			(xy 109.22 102.87) (xy 87.63 102.87)
-		)
-		(stroke
-			(width 0)
-			(type default)
-		)
-	)
-	(wire
-		(pts
-			(xy 175.26 100.33) (xy 204.47 100.33)
-		)
-		(stroke
-			(width 0)
-			(type default)
-		)
-	)
-	(wire
-		(pts
-			(xy 144.78 123.19) (xy 144.78 124.46)
-		)
-		(stroke
-			(width 0)
-			(type default)
-		)
-	)
-	(wire
-		(pts
-			(xy 144.78 124.46) (xy 142.24 124.46)
-		)
-		(stroke
-			(width 0)
-			(type default)
-		)
-	)
-	(wire
-		(pts
-			(xy 204.47 97.79) (xy 175.26 97.79)
-		)
-		(stroke
-			(width 0)
-			(type default)
-		)
-	)
-	(wire
-		(pts
-			(xy 175.26 105.41) (xy 177.8 105.41)
-		)
-		(stroke
-			(width 0)
-			(type default)
-		)
-	)
-	(wire
-		(pts
-			(xy 129.54 124.46) (xy 125.73 124.46)
-		)
-		(stroke
-			(width 0)
-			(type default)
-		)
-	)
-	(wire
-		(pts
-			(xy 204.47 100.33) (xy 204.47 101.6)
-		)
-		(stroke
-			(width 0)
-			(type default)
-		)
-	)
-	(wire
-		(pts
-			(xy 142.24 50.8) (xy 142.24 54.61)
-		)
-		(stroke
-			(width 0)
-			(type default)
-		)
-	)
-	(wire
-		(pts
-			(xy 87.63 100.33) (xy 87.63 102.87)
-		)
-		(stroke
-			(width 0)
-			(type default)
-		)
-	)
-	(wire
-		(pts
-			(xy 177.8 105.41) (xy 193.04 105.41)
-		)
-		(stroke
-			(width 0)
-			(type default)
-		)
-	)
-	(wire
-		(pts
-			(xy 129.54 132.08) (xy 129.54 133.35)
-		)
-		(stroke
-			(width 0)
-			(type default)
-		)
-	)
-	(wire
-		(pts
-			(xy 33.02 30.48) (xy 45.72 30.48)
-		)
-		(stroke
-			(width 0)
-			(type default)
-		)
-	)
-	(wire
-		(pts
 			(xy 139.7 123.19) (xy 139.7 124.46)
 		)
@@
 	(wire
 		(pts
-			(xy 139.7 50.8) (xy 139.7 54.61)
+			(xy 139.7 45.72) (xy 139.7 54.61)
 		)
 		(stroke
@@
 		(pts
 			(xy 142.24 124.46) (xy 142.24 125.73)
+		)
+		(stroke
+			(width 0)
+			(type default)
+		)
+	)
+	(wire
+		(pts
+			(xy 154.94 49.53) (xy 165.1 49.53)
 		)
 		(stroke
@@
 		)
 	)
+	(text "SPRAWDZIĆ CZY JEST OK (rezystor) I CZY MUSI BYC NA MISO (napewno \nnie ale z jakiegos powodu tak jest teraz fizycznie)"
+		(exclude_from_sim no)
+		(at 188.722 42.164 0)
+		(effects
+			(font
+				(size 1.27 1.27)
+			)
+		)
+	)
 	(text "I2C address: (old)\n1101000\n0x68"
 		(exclude_from_sim no)
@@
 	)
 	(label "3,3V_imu"
+		(at 157.48 49.53 0)
+		(fields_autoplaced yes)
+		(effects
+			(font
+				(size 1.27 1.27)
+			)
+			(justify left bottom)
+		)
+	)
+	(label "3,3V_imu"
 		(at 36.83 30.48 0)
 		(fields_autoplaced yes)
@@
 	(hierarchical_label "MOSI_imu"
 		(shape input)
-		(at 139.7 50.8 90)
+		(at 139.7 45.72 90)
 		(fields_autoplaced yes)
 		(effects
@@
 	(hierarchical_label "CS_imu"
 		(shape input)
-		(at 144.78 50.8 90)
+		(at 144.78 45.72 90)
 		(fields_autoplaced yes)
 		(effects
@@
 	(hierarchical_label "SCK_imu"
 		(shape input)
-		(at 142.24 50.8 90)
+		(at 142.24 45.72 90)
 		(fields_autoplaced yes)
 		(effects
@@
 					(unit 1)
 				)
+			)
+		)
+	)
+	(symbol
+		(lib_id "Device:R")
+		(at 151.13 49.53 90)
+		(unit 1)
+		(exclude_from_sim no)
+		(in_bom yes)
+		(on_board yes)
+		(dnp no)
+		(fields_autoplaced yes)
+		(property "Reference" "R17"
+			(at 151.13 43.18 90)
+			(effects
+				(font
+					(size 1.27 1.27)
+				)
+			)
+		)
+		(property "Value" "10k"
+			(at 151.13 45.72 90)
+			(effects
+				(font
+					(size 1.27 1.27)
+				)
+			)
+		)
+		(property "Footprint" "Resistor_SMD:R_0603_1608Metric"
+			(at 151.13 51.308 90)
+			(effects
+				(font
+					(size 1.27 1.27)
+				)
+				(hide yes)
+			)
+		)
+		(property "Datasheet" "~"
+			(at 151.13 49.53 0)
+			(effects
+				(font
+					(size 1.27 1.27)
+				)
+				(hide yes)
+			)
+		)
+		(property "Description" "Resistor"
+			(at 151.13 49.53 0)
+			(effects
+				(font
+					(size 1.27 1.27)
+				)
+				(hide yes)
+			)
+		)
+		(pin "2"
+		)
+		(pin "1"
+		)
+		(instances
+			(project ""
+				(path "/ade9c7e9-87ec-416b-ada9-3e894081f6ea/9006e8d8-741e-44dd-bd3c-e3e388e000b6"
+					(reference "R17")
+					(unit 1)
+				)
