File: kontroler_lotu.kicad_pcb (KiCad board)
At the start: 2 copper layers, 70 x 69.7 mm, 73 parts, among them IC1 ICM-42688-P, IC3 FM24CL16B-GTR, J1 input_voltage, J10 BOOT0 STATE, J11 GPS, J12 pololu_LV, J13 pololu_HV, J14 690-005-299-043, J15 MCU_EXTRA2, J16 MCU_EXTRA3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

Commit message: Zamieniono konwerter napięć na SMD. Zaktualizowano projekt PCB. Usunięto błedy - zostało część ostrzeżeń dotyczących nakładających się silk.
Parts:
- removed J12: pololu_LV, Connector_PinHeader_2.54mm:PinHeader_1x05_P2.54mm_Vertical
- removed J13: pololu_HV, Connector_PinHeader_2.54mm:PinHeader_1x05_P2.54mm_Vertical
- added C24: 47uF, Capacitor_Tantalum_SMD:CP_EIA-3528-12_Kemet-T, F.Cu at (120.8, 118.7)
- added C25: 100nF, Capacitor_SMD:C_0603_1608Metric, F.Cu at (126.5, 119.5)
- added C26: 22uF, Capacitor_Tantalum_SMD:CP_EIA-3528-12_Kemet-T, F.Cu at (124.8, 112.4)
- added C27: 100nF, Capacitor_SMD:C_0603_1608Metric, F.Cu at (123.8, 114.9)
- added C28: 0.1uF, Capacitor_SMD:C_0603_1608Metric, F.Cu at (116.7, 79.0)
- added C29: 0.1uF, Capacitor_SMD:C_0603_1608Metric, F.Cu at (116.5, 68.3)
- added D5: RED LED [Polarity Fault], LED_SMD:LED_0805_2012Metric, F.Cu at (103.2, 120.0)
- added FB1: BLM21PG121BH1D, Inductor_SMD:L_0805_2012Metric_Pad1.15x1.40mm_HandSolder, F.Cu at (124.6, 117.6)
- added Q1: IRML9301TRPbF, Package_TO_SOT_SMD:SOT-23, F.Cu at (109.9, 120.1)
- added Q2: 2N3906, Package_TO_SOT_THT:TO-92L_Inline, F.Cu at (108.0, 116.5)
- added Q3: 2N3906, Package_TO_SOT_THT:TO-92L_Inline, F.Cu at (111.8, 114.1)
- added R12: 10k, Resistor_SMD:R_0603_1608Metric, F.Cu at (105.9, 111.0)
- added R13: 10k, Resistor_SMD:R_0603_1608Metric, F.Cu at (108.7, 111.0)
- added R14: 1k, Resistor_SMD:R_0603_1608Metric, F.Cu at (105.0, 119.8)
- added TVS1: SMBJ5.0A, Diode_SMD:D_SMB_Handsoldering, F.Cu at (116.9, 117.6)
- added U4: TXS0108EPW, Package_SO:TSSOP-20_4.4x6.5mm_P0.65mm, F.Cu at (119.6, 73.5)
- moved TP2 31.2 mm to (132.8, 96.3)
- moved J1 28.3 mm to (97.8, 119.7), turned to 90 degrees
- moved H4 4.11 mm to (132.0, 119.3)
- moved H2 4.11 mm to (73.0, 119.3)
- moved J14 3.70 mm to (83.4, 123.3)
Connections:
- IC1 pad 1: /IMU/SCK_imu -> /IMU/MISO_imu
- IC1 pad 13: /IMU/MISO_imu -> /IMU/SCK_imu
- J1 pad 2: /+5v_supply -> Net-(D5-K)
Routing:
- net Net-(Q1-S): track 0.00 -> 20.1 mm
- net Net-(D5-K): track 0.00 -> 18.8 mm
- net Net-(Q1-G): track 0.00 -> 14.1 mm, vias 0 -> 1
- net Net-(Q2-B): track 0.00 -> 12.6 mm
- net /+5v_supply: track 153.1 -> 158.2 mm, vias 2 -> 3
- net /USB/DP: track 9.72 -> 13.4 mm
- net /USB/DN: track 9.68 -> 13.4 mm
- net /USB/shield: track 32.3 -> 35.6 mm
- net Net-(D5-A): track 0.00 -> 1.84 mm
- net /IMU/SCK_imu: track 4.49 -> 5.98 mm, vias 0 -> 2
- net /STM32/outlet_rx: track 28.8 -> 29.7 mm, vias 1 -> 2
- net Net-(J6-Pin_2): track 15.1 -> 14.4 mm, vias 0 -> 1
- net /IMU/MISO_imu: track 4.08 -> 4.70 mm, vias 2 -> 0
- net /IMU/CS_imu: track 6.70 -> 7.24 mm
- net Net-(J6-Pin_3): track 15.1 -> 14.6 mm, vias 0 -> 1
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Other:
- board size 70 x 69.7 mm -> 70 x 73.8 mm
- board text added: "Kontroler Lotu V1.1"
- board text added: "MKL Styczeń 2026"
- board text removed: "Kontroler Lotu V1.0"
- board text removed: "MKL Lipiec 2025"
- board text removed: "Pololu"

Commit message: dodano komentarze do projektu
Parts:
- added J12: raw_input_voltage, Connector_PinSocket_2.54mm:PinSocket_1x02_P2.54mm_Vertical, F.Cu at (131.9, 110.1)
- added R16: 10k, Resistor_SMD:R_0603_1608Metric, F.Cu at (83.1, 66.4)
- added R17: 10k, Resistor_SMD:R_0603_1608Metric, B.Cu at (94.3, 87.3)
Connections:
- J14 pad 6: /USB/shield -> (no net)
- J14 pad 7: /USB/shield -> (no net)
- J14 pad 8: /USB/shield -> (no net)
- J14 pad 9: /USB/shield -> (no net)
Routing:
- net /IMU/3,3V_imu: track 193.9 -> 207.4 mm
- net /+5v_supply: track 158.2 -> 167.0 mm
- net Net-(J18-Pin_1): track 25.5 -> 29.5 mm
Other:
- board text added: "fault"
- board text added: "supp2"
