File: kontroler_lotu.kicad_sch (KiCad schematic)
At the start: 4 parts

Commit message: Dodano układ wejściowy dla zasilania. Nie symulowano całości.
Other:
- added sheet Volt Supp (volt_supp.kicad_sch)
Changed lines of the file:
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@@
+	(wire
+		(pts
+			(xy 161.29 58.42) (xy 171.45 58.42)
+		)
+		(stroke
+			(width 0)
+			(type default)
+		)
+	)
 	(wire
 		(pts
@@
 	(label "+5v_supply"
 		(at 176.53 116.84 0)
+		(fields_autoplaced yes)
+		(effects
+			(font
+				(size 1.27 1.27)
+			)
+			(justify left bottom)
+		)
+	)
+	(label "+5v_supply"
+		(at 162.56 58.42 0)
 		(fields_autoplaced yes)
 		(effects
@@
 				)
 			)
+		)
+	)
+	(sheet
+		(at 121.92 48.26)
+		(size 39.37 13.335)
+		(fields_autoplaced yes)
+		(stroke
+			(width 0.1524)
+			(type solid)
+		)
+		(fill
+			(color 0 0 0 0.0000)
+		)
+		(property "Sheetname" "Volt Supp"
+			(at 121.92 47.5484 0)
+			(effects
+				(font
+					(size 1.27 1.27)
+				)
+				(justify left bottom)
+			)
+		)
+		(property "Sheetfile" "volt_supp.kicad_sch"
+			(at 121.92 62.1796 0)
+			(effects
+				(font
+					(size 1.27 1.27)
+				)
+				(justify left top)
+			)
+		)
+		(pin "+5v_supply" output
+			(at 161.29 58.42 0)
+			(effects
+				(font
+					(size 1.27 1.27)
+				)
+				(justify right)
+			)
+		)
+		(instances
+			(project "kontroler_lotu"
+				(path "/ade9c7e9-87ec-416b-ada9-3e894081f6ea"
+					(page "6")
+				)
+			)

Commit message: dodano komentarze do projektu
Changed lines of the file:
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@@
+		)
+	)
+	(text_box "komentarze do poprawy w tym projekcie:\n1) Footprint MOSFET jest nieprawidłowy\n2) Zrobić socket na programator np. 4x2 konektor"
+		(exclude_from_sim no)
+		(at 18.415 18.415 0)
+		(size 52.07 31.115)
+		(stroke
+			(width 0)
+			(type default)
+		)
+		(fill
+			(type none)
+		)
+		(effects
+			(font
+				(size 1.27 1.27)
+			)
+			(justify left top)
 		)
 	)
